File: NANOetFETs/MainControll/MainControll.sch (EAGLE design)
At the start: 17 parts

Commit message: 1st prototype
Parts:
- added JP1: (no value), pinhead:PINHD-1X4
- FET_AIRPUMP, FET_COLLECTPUMP, FET_VALVE, FET_WATERPUMP: value IRF740 -> 2SK2232; device transistor-power:IRF740 -> Transistor-FET:2SK2232
Connections:
- new net N$1: JP1.3, U$2.RX1
- new net N$2: JP1.2, U$2.TX0
- net +12V: now also JP1.1
- net GND: now also JP1.4
Changed lines of the file:
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@@
 </classes>
 <parts>
-<part name="FET_VALVE" library="transistor-power" library_urn="urn:adsk.eagle:library:400" deviceset="IRF740" device="" package3d_urn="urn:adsk.eagle:package:29484/3"/>
-<part name="FET_WATERPUMP" library="transistor-power" library_urn="urn:adsk.eagle:library:400" deviceset="IRF740" device="" package3d_urn="urn:adsk.eagle:package:29484/3"/>
-<part name="FET_COLLECTPUMP" library="transistor-power" library_urn="urn:adsk.eagle:library:400" deviceset="IRF740" device="" package3d_urn="urn:adsk.eagle:package:29484/3"/>
+<part name="FET_VALVE" library="Transistor-FET" library_urn="urn:adsk.eagle:library:11887002" deviceset="2SK2232" device="" package3d_urn="urn:adsk.eagle:package:8089444/1"/>
+<part name="FET_WATERPUMP" library="Transistor-FET" library_urn="urn:adsk.eagle:library:11887002" deviceset="2SK2232" device="" package3d_urn="urn:adsk.eagle:package:8089444/1"/>
+<part name="FET_COLLECTPUMP" library="Transistor-FET" library_urn="urn:adsk.eagle:library:11887002" deviceset="2SK2232" device="" package3d_urn="urn:adsk.eagle:package:8089444/1"/>
 <part name="TERMINAL_AIRPUMP" library="terminal_block_5.08mm" deviceset="TERMINAL_BLOCK_5.08MM" device=""/>
 <part name="TERMINAL_VALVE" library="terminal_block_5.08mm" deviceset="TERMINAL_BLOCK_5.08MM" device=""/>
@@
 <part name="SW_LED" library="pinhead" library_urn="urn:adsk.eagle:library:325" deviceset="PINHD-1X5" device="" package3d_urn="urn:adsk.eagle:package:22469/2"/>
 <part name="SW" library="pinhead" library_urn="urn:adsk.eagle:library:325" deviceset="PINHD-1X5" device="" package3d_urn="urn:adsk.eagle:package:22469/2"/>
-<part name="FET_AIRPUMP" library="transistor-power" library_urn="urn:adsk.eagle:library:400" deviceset="IRF740" device="" package3d_urn="urn:adsk.eagle:package:29484/3"/>
+<part name="FET_AIRPUMP" library="Transistor-FET" library_urn="urn:adsk.eagle:library:11887002" deviceset="2SK2232" device="" package3d_urn="urn:adsk.eagle:package:8089444/1"/>
 <part name="U$1" library="terminal_block_5.08mm" deviceset="TERMINAL_BLOCK_5.08MM" device=""/>
 <part name="GND1" library="supply1" library_urn="urn:adsk.eagle:library:371" deviceset="GND" device=""/>
@@
 <part name="C1" library="rcl" library_urn="urn:adsk.eagle:library:334" deviceset="CPOL-EU" device="E2.5-5" package3d_urn="urn:adsk.eagle:package:23344/1"/>
 <part name="U$2" library="Arduino-clone" deviceset="NANO_DIL_RECEPTOR" device=""/>
+<part name="JP1" library="pinhead" library_urn="urn:adsk.eagle:library:325" deviceset="PINHD-1X4" device="" package3d_urn="urn:adsk.eagle:package:22407/2"/>
+<part name="GND6" library="supply1" library_urn="urn:adsk.eagle:library:371" deviceset="GND" device=""/>
+<part name="P+6" library="supply1" library_urn="urn:adsk.eagle:library:371" deviceset="+12V" device=""/>
 </parts>
 <sheets>
@@
 </instance>
 <instance part="U$2" gate="G$1" x="35.56" y="38.1" smashed="yes"/>
+<instance part="JP1" gate="A" x="60.96" y="22.86" smashed="yes" rot="R180">
+<attribute name="NAME" x="67.31" y="14.605" size="1.778" layer="95" rot="R180"/>
+<attribute name="VALUE" x="67.31" y="30.48" size="1.778" layer="96" rot="R180"/>
+</instance>
+<instance part="GND6" gate="1" x="71.12" y="20.32" smashed="yes">
+<attribute name="VALUE" x="68.58" y="17.78" size="1.778" layer="96"/>
+</instance>
+<instance part="P+6" gate="1" x="55.88" y="17.78" smashed="yes">
+<attribute name="VALUE" x="53.34" y="12.7" size="1.778" layer="96" rot="R90"/>
+</instance>
 </instances>
 <busses>
@@
 <pinref part="U$2" gate="G$1" pin="GND"/>
 </segment>
+<segment>
+<pinref part="JP1" gate="A" pin="4"/>
+<wire x1="63.5" y1="25.4" x2="71.12" y2="25.4" width="0.1524" layer="91"/>
+<wire x1="71.12" y1="25.4" x2="71.12" y2="22.86" width="0.1524" layer="91"/>
+<pinref part="GND6" gate="1" pin="GND"/>
+</segment>
 </net>
 <net name="+5V" class="0">
@@
 <junction x="96.52" y="81.28"/>
 </segment>
+<segment>
+<pinref part="P+6" gate="1" pin="+12V"/>
+<pinref part="JP1" gate="A" pin="1"/>
+<wire x1="55.88" y1="15.24" x2="63.5" y2="15.24" width="0.1524" layer="91"/>
+<wire x1="63.5" y1="15.24" x2="63.5" y2="17.78" width="0.1524" layer="91"/>
+</segment>
 </net>
 <net name="VALVE" class="0">
@@
 </segment>
 </net>
+<net name="N$1" class="0">
+<segment>
+<pinref part="U$2" gate="G$1" pin="RX1"/>
+<pinref part="JP1" gate="A" pin="3"/>
+<wire x1="50.8" y1="22.86" x2="63.5" y2="22.86" width="0.1524" layer="91"/>
+</segment>
+</net>
+<net name="N$2" class="0">
+<segment>
+<pinref part="U$2" gate="G$1" pin="TX0"/>
+<pinref part="JP1" gate="A" pin="2"/>
+<wire x1="50.8" y1="20.32" x2="63.5" y2="20.32" width="0.1524" layer="91"/>
+</segment>
+</net>
