File: NANOetFETs/MainControll/MainControll.brd (EAGLE design)
At the start: 85 x 55 mm, 18 parts

Commit message: release
Routing:
- net SW2: track 88.7 -> 84.6 mm
Other:
- board text added: "MainControl - 2022/1"
- board text removed: "失禁研究会MainControl - 2022/1"
Changed lines of the file:
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@@
 <setting verticaltext="up"/>
 </settings>
-<grid distance="1" unitdist="mm" unit="mm" style="lines" multiple="1" display="yes" altdistance="1" altunitdist="mil" altunit="mil"/>
+<grid distance="3" unitdist="mil" unit="mil" style="lines" multiple="1" display="yes" altdistance="1" altunitdist="mil" altunit="mil"/>
 <layers>
 <layer number="1" name="Top" color="4" fill="1" visible="yes" active="yes"/>
@@
 <wire x1="2.5" y1="0" x2="0" y2="2.5" width="0.0762" layer="20" curve="-90" grouprefs="PCB"/>
 <wire x1="85" y1="2.5" x2="82.5" y2="0" width="0.0762" layer="20" curve="-90" grouprefs="PCB"/>
-<text x="6.985" y="52.451" size="1.778" layer="25" grouprefs="PCB">失禁研究会MainControl - 2022/1</text>
+<text x="8.3566" y="52.451" size="1.778" layer="25" grouprefs="PCB">MainControl - 2022/1</text>
 <rectangle x1="8.6002" y1="40.4478" x2="8.7526" y2="40.6002" layer="25"/>
 <rectangle x1="9.5146" y1="40.4478" x2="9.667" y2="40.6002" layer="25"/>
@@
 </element>
 <element name="FET_AIRPUMP" library="Transistor-FET" library_urn="urn:adsk.eagle:library:11887002" package="TO220" package3d_urn="urn:adsk.eagle:package:8089444/1" value="2SK2232" x="64.77" y="46.99" smashed="yes" rot="R90" grouprefs="PCB">
-<attribute name="NAME" x="62.468" y="41.2662" size="1.27" layer="25" ratio="10" rot="R180"/>
-<attribute name="VALUE" x="65.278" y="51.308" size="1.27" layer="27" ratio="10" rot="R180"/>
+<attribute name="NAME" x="50.0032" y="40.2678" size="1.27" layer="25" ratio="10"/>
+<attribute name="VALUE" x="57.785" y="50.038" size="1.27" layer="27" ratio="10"/>
 </element>
 <element name="FET_COLLECTPUMP" library="Transistor-FET" library_urn="urn:adsk.eagle:library:11887002" package="TO220" package3d_urn="urn:adsk.eagle:package:8089444/1" value="2SK2232" x="64.77" y="21.59" smashed="yes" rot="R90" grouprefs="PCB">
-<attribute name="NAME" x="67.818" y="15.8902" size="1.27" layer="25" ratio="10" rot="R180"/>
-<attribute name="VALUE" x="65.278" y="26.035" size="1.27" layer="27" ratio="10" rot="R180"/>
+<attribute name="NAME" x="49.9872" y="14.8184" size="1.27" layer="25" ratio="10"/>
+<attribute name="VALUE" x="57.8612" y="24.638" size="1.27" layer="27" ratio="10"/>
 </element>
 <element name="FET_VALVE" library="Transistor-FET" library_urn="urn:adsk.eagle:library:11887002" package="TO220" package3d_urn="urn:adsk.eagle:package:8089444/1" value="2SK2232" x="64.77" y="34.29" smashed="yes" rot="R90" grouprefs="PCB">
-<attribute name="NAME" x="59.817" y="28.9052" size="1.27" layer="25" ratio="10" rot="R180"/>
-<attribute name="VALUE" x="65.405" y="38.608" size="1.27" layer="27" ratio="10" rot="R180"/>
+<attribute name="NAME" x="50.0634" y="27.4828" size="1.27" layer="25" ratio="10"/>
+<attribute name="VALUE" x="57.8104" y="37.4396" size="1.27" layer="27" ratio="10"/>
 </element>
 <element name="FET_WATERPUMP" library="Transistor-FET" library_urn="urn:adsk.eagle:library:11887002" package="TO220" package3d_urn="urn:adsk.eagle:package:8089444/1" value="2SK2232" x="64.77" y="8.89" smashed="yes" rot="R90" grouprefs="PCB">
-<attribute name="NAME" x="65.826" y="3.0242" size="1.27" layer="25" ratio="10" rot="R180"/>
-<attribute name="VALUE" x="65.278" y="13.335" size="1.27" layer="27" ratio="10" rot="R180"/>
+<attribute name="NAME" x="49.998" y="2.005" size="1.27" layer="25" ratio="10"/>
+<attribute name="VALUE" x="57.8612" y="11.9634" size="1.27" layer="27" ratio="10"/>
 </element>
 <element name="R1" library="rcl" library_urn="urn:adsk.eagle:library:334" package="0204/5" package3d_urn="urn:adsk.eagle:package:23488/1" value="103" x="29.21" y="41.91" smashed="yes" rot="R270" grouprefs="PCB">
@@
 <contactref element="U$2" pad="D11"/>
 <wire x1="6.35" y1="24.13" x2="6.35" y2="36.83" width="1.27" layer="1" grouprefs="PCB"/>
-<wire x1="42.545" y1="24.13" x2="6.35" y2="24.13" width="1.27" layer="1" grouprefs="PCB"/>
-<wire x1="44.45" y1="22.225" x2="42.545" y2="24.13" width="1.27" layer="1" grouprefs="PCB"/>
-<wire x1="44.45" y1="4.445" x2="44.45" y2="22.225" width="1.27" layer="1" grouprefs="PCB"/>
-<wire x1="28.575" y1="4.445" x2="44.45" y2="4.445" width="1.27" layer="1" grouprefs="PCB"/>
+<wire x1="6.35" y1="24.13" x2="42.545" y2="24.13" width="1.27" layer="1" grouprefs="PCB"/>
 <wire x1="26.67" y1="6.35" x2="28.575" y2="4.445" width="1.27" layer="1" grouprefs="PCB"/>
 <wire x1="26.67" y1="7.112" x2="26.67" y2="6.35" width="1.27" layer="1" grouprefs="PCB"/>
+<wire x1="28.575" y1="4.445" x2="37.8968" y2="4.445" width="1.27" layer="1"/>
+<wire x1="44.1198" y1="10.668" x2="37.8968" y2="4.445" width="1.27" layer="1"/>
+<wire x1="42.545" y1="24.13" x2="44.1198" y2="22.5552" width="1.27" layer="1"/>
+<wire x1="44.1198" y1="22.5552" x2="44.1198" y2="10.668" width="1.27" layer="1"/>
 </signal>
 <signal name="N$11">
@@
 <wire x1="71.755" y1="19.685" x2="71.12" y2="19.05" width="1.27" layer="1" grouprefs="PCB"/>
 <wire x1="75.565" y1="19.685" x2="71.755" y2="19.685" width="1.27" layer="1" grouprefs="PCB"/>
-<wire x1="78.74" y1="22.86" x2="75.565" y2="19.685" width="1.27" layer="1" grouprefs="PCB"/>
-<wire x1="81.28" y1="22.86" x2="78.74" y2="22.86" width="1.27" layer="1" grouprefs="PCB"/>
-<wire x1="82.55" y1="24.13" x2="81.28" y2="22.86" width="1.27" layer="1" grouprefs="PCB"/>
-<wire x1="82.55" y1="38.1" x2="82.55" y2="24.13" width="1.27" layer="1" grouprefs="PCB"/>
-<wire x1="73.66" y1="38.1" x2="82.55" y2="38.1" width="1.27" layer="1" grouprefs="PCB"/>
-<wire x1="71.755" y1="40.005" x2="73.66" y2="38.1" width="1.27" layer="1" grouprefs="PCB"/>
+<wire x1="78.5876" y1="22.7076" x2="75.565" y2="19.685" width="1.27" layer="1" grouprefs="PCB"/>
+<wire x1="81.8896" y1="22.7076" x2="78.5876" y2="22.7076" width="1.27" layer="1" grouprefs="PCB"/>
 <wire x1="31.115" y1="40.005" x2="71.755" y2="40.005" width="1.27" layer="1" grouprefs="PCB"/>
 <wire x1="29.845" y1="41.275" x2="31.115" y2="40.005" width="1.27" layer="1" grouprefs="PCB"/>
 <wire x1="26.035" y1="41.275" x2="29.845" y2="41.275" width="1.27" layer="1" grouprefs="PCB"/>
 <wire x1="24.13" y1="39.37" x2="26.035" y2="41.275" width="1.27" layer="1" grouprefs="PCB"/>
+<wire x1="74.041" y1="37.719" x2="81.3054" y2="37.719" width="1.27" layer="1"/>
+<wire x1="81.3054" y1="37.719" x2="83.1342" y2="35.8902" width="1.27" layer="1"/>
+<wire x1="71.755" y1="40.005" x2="74.041" y2="37.719" width="1.27" layer="1" grouprefs="PCB"/>
+<wire x1="83.1342" y1="35.8902" x2="83.1342" y2="23.9522" width="1.27" layer="1"/>
+<wire x1="83.1342" y1="23.9522" x2="81.8896" y2="22.7076" width="1.27" layer="1"/>
 </signal>
 <signal name="WATPUMP">
